File: Ethernet.kicad_sch (KiCad schematic)
At the start: 6 parts, among them T401 7498111120AR, U401 TPD4EUSB30, U402 TPD4EUSB30

Commit message: Finished Everything
Parts:
- removed T401: 7498111120AR, Ethernet:7498111120AR, symbol Connector:WE-RJ45_7498111120AR
- added U1: MagJack-A70-112-331N126, CM5IO:TRJG0926HENL, symbol CM5IO:MagJack-A70-112-331N126
Connections:
- net +3V3_PI: now also U1.15 (LEDY_A), U1.17 (LEDG_A)
- net ETH_C.TRD0_N: now also U1.2 (TRD0-)
- net ETH_C.TRD0_P: now also U1.1 (TRD0+)
- net ETH_C.TRD1_N: now also U1.6 (TRD1-)
- net ETH_C.TRD1_P: now also U1.3 (TRD1+)
- net ETH_C.TRD2_N: now also U1.8 (TRD2-)
- net ETH_C.TRD2_P: now also U1.7 (TRD2+)
- net ETH_C.TRD3_N: now also U1.10 (TRD3-)
- net ETH_C.TRD3_P: now also U1.9 (TRD3+)
- net GND: now also U1.19 (SHIELD), U1.20 (SHIELD)
- net at R402.2: now also U1.16 (LEDY_K)
- net at R401.2: now also U1.18 (LEDG_K)
- net at C401.1: now also U1.4 (CT), U1.5 (CT)
- no-connect marks 0 -> 4
Other:
- note removed: "Ethernet POE Protection"
- moved on the sheet: C401, R401, R402
