File: MainPCB.kicad_pcb (KiCad board)
At the start: 6 copper layers, 128 x 89.5 mm, 108 parts, among them IC1 VNH7070ASTR, IC2 VNH7070ASTR, IC3 VNH7070ASTR, IC4 VNH7070ASTR, IC5 VNH7070ASTR, J1 Conn_01x06, J10 Conn_01x02, J101 TYPEC-305-ACP16H458, J11 Conn_01x03, J20 Conn_01x02_Pin, J3 Conn_01x03_Pin, J4 Conn_01x02, J5 Screw_Terminal_01x02, J501 GT-HD001B-CNNG1, J6 Conn_01x04_Pin, J7 Conn_01x04_Pin, J8 Conn_01x02, J802 Conn_01x22_Female, J9 Conn_01x06_Pin, M1 Motor_DC, M2 Motor_DC, M3 Motor_DC, M4 Motor_DC, M5 Motor_DC, SW1 SW_DPST_x2, SW2 SW_DPST_x2, U1 MagJack-A70-112-331N126, U10 N channel, U12 Teensy4.1, U21 V_Regulator3.3v, U22 V_Regulator5v, U4 BNO055, U401 TPD4EUSB30, U402 TPD4EUSB30, U405 STMPS2151STR, U602 SN74LVC1G14DBVR, U701 AP22653W6

Commit message: Finished
Routing:
- net GND: track 0.00 -> 240.1 mm, vias 0 -> 48
- net /CM5/nLED_ACTIVITY: track 0.00 -> 110.8 mm, vias 0 -> 2
- net 12V: track 260.6 -> 368.9 mm, vias 13 -> 14
- net /CM5/ETH_nLED_ACTIVITY: track 1.83 -> 109.1 mm, vias 2 -> 5
- net PWM-LIDAR: track 28.5 -> 127.8 mm, vias 3 -> 5
- net RX->TX - LIDAR: track 37.7 -> 136.7 mm
- net /CM5/nLED_SPEED_100_1000: track 1.38 -> 92.7 mm, vias 2 -> 5
- net RX3->TX: track 0.00 -> 74.8 mm, vias 0 -> 3
- net TX3->RX: track 0.00 -> 70.9 mm, vias 0 -> 4
- net /CM5/PI_nLED_PWR: track 5.87 -> 70.1 mm
- net /CM5/DPHY0_P.D0_P: track 130.3 -> 70.1 mm
- net /CC2: track 4.83 -> 62.5 mm
- net /CM5/CAM_GPIO1: track 13.2 -> 70.7 mm
- net /CC1: track 0.00 -> 56.2 mm, vias 0 -> 2
- net /CM5/HDMI_PI.D2_P: track 113.8 -> 58.7 mm, vias 4 -> 2
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
Commit message: updated some traces
Parts:
- moved C601 1.13 mm to (134.4, 123.9)
Routing:
- net 5V: track 565.2 -> 514.3 mm
- net 12V: track 368.9 -> 345.8 mm
- net PWM-LIDAR: track 127.8 -> 119.6 mm
- net Net-(IC1-OUT_B_1): track 61.7 -> 59.2 mm
- net Net-(IC1-OUT_A_1): track 77.1 -> 75.4 mm
- net 3.3V: track 574.1 -> 574.6 mm
- net GND: track 240.1 -> 240.0 mm, vias 48 -> 81
