File: HDMI.kicad_sch (KiCad schematic)
At the start: 7 parts, among them J501 GT-HD001B-CNNG1, U405 STMPS2151STR

Commit message: Made changes to placement and HDMI is now vertical
Parts:
- J501: footprint CM5IO:EDAC 690-019-298-412 -> HDMI-Conn:PHOENIX_1332073; Current Connector (none) -> https://www.digikey.com/en/products/detail/phoenix-contact/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
Changed lines of the file:
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@@
 			)
 		)
-		(property "Footprint" "CM5IO:EDAC 690-019-298-412"
+		(property "Footprint" "HDMI-Conn:PHOENIX_1332073"
 			(at 212.725 78.74 0)
 			(hide yes)
@@
 			(at 212.09 78.74 0)
 			(hide yes)
+			(show_name no)
+			(do_not_autoplace no)
+			(effects
+				(font
+					(size 1.27 1.27)
+				)
+			)
+		)
+		(property "Current Connector" "https://www.digikey.com/en/products/detail/phoenix-contact/1332073/17940320"
+			(at 212.09 78.74 0)
+			(hide yes)
