File: _restore_backup_2026-05-25T19-17-20-350/MainPCB.kicad_pcb (KiCad board)
At the start: 6 copper layers, 128 x 89.5 mm, 112 parts, among them IC1 VNH7070ASTR, IC2 VNH7070ASTR, IC3 VNH7070ASTR, IC4 VNH7070ASTR, IC5 VNH7070ASTR, J1 Conn_01x06, J10 Conn_01x02, J101 TYPEC-305-ACP16H458, J11 Conn_01x03, J20 Conn_01x02_Pin, J3 Conn_01x03_Pin, J4 Conn_01x02, J5 Screw_Terminal_01x02, J501 GT-HD001B-CNNG1, J6 Conn_01x04_Pin, J7 Conn_01x04_Pin, J8 Conn_01x02, J802 Conn_01x22_Female, J9 Conn_01x06_Pin, M1 Motor_DC, M2 Motor_DC, M3 Motor_DC, M4 Motor_DC, M5 Motor_DC, SW1 SW_DPST_x2, SW2 SW_DPST_x2, U1 MagJack-A70-112-331N126, U10 N channel, U12 Teensy4.1, U21 V_Regulator3.3v, U22 V_Regulator5v, U4 BNO055, U401 TPD4EUSB30, U402 TPD4EUSB30, U405 STMPS2151STR, U602 SN74LVC1G14DBVR, U701 AP22653W6

Commit message: Changes
Parts:
- removed R19: 10k, Capacitor_SMD:C_0805_2012Metric_Pad1.18x1.45mm_HandSolder
- removed REF** (x2): Adafruit TDK InvenSense ICM-20948 9-DoF IMU, Custom:Adafruit TDK InvenSense ICM-20948 9-DoF IMU
- removed SW2: SW_DPST_x2, Custom:Latch-Switch
Connections:
- U12 pad 30: Start/Stop -> unconnected-(U12-38_CS1_IN1-Pad30)
Routing:
- net Start/Stop: track 81.0 -> 0.00 mm, vias 1 -> 0
- net DIR5A: track 104.3 -> 119.9 mm
- net 3.3V: track 351.1 -> 340.1 mm
- net GND: track 224.5 -> 219.7 mm
- net RX7 -> TX: track 99.8 -> 98.5 mm
- net SDA2: track 122.1 -> 123.1 mm
