File: _restore_backup_2026-05-25T19-17-20-350/MainPCB.kicad_sch (KiCad schematic)
At the start: 76 parts, among them IC1 VNH7070ASTR, IC2 VNH7070ASTR, IC3 VNH7070ASTR, IC4 VNH7070ASTR, IC5 VNH7070ASTR, J1 Conn_01x06, J10 Conn_01x02, J101 TYPEC-305-ACP16H458, J11 Conn_01x03, J20 Conn_01x02_Pin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

Commit message: Changes
Parts:
- SW2: footprint Custom:Latch-Switch -> SlideSW:SPDT_OS102011_CNK
Changed lines of the file:
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@@
 			)
 		)
-		(property "Footprint" "Custom:Latch-Switch"
+		(property "Footprint" "SlideSW:SPDT_OS102011_CNK"
 			(at 132.08 146.05 0)
 			(hide yes)
